File: lichtenprog.sch (KiCad schematic (older format))
At the start: 16 parts, among them J1 USB_B_Mini, J2 Conn_01x06, U1 AMS1117-3.3, U2 CP2102N-A01-GQFN28

Commit message: rev 2 schematic and PCB do-over
Parts:
- removed J2: Conn_01x06, Connector_PinHeader_2.54mm:PinHeader_1x06_P2.54mm_Vertical, symbol Connector_Generic:Conn_01x06
- added C5: 2.2u, Capacitor_SMD:C_0603_1608Metric_Pad1.05x0.95mm_HandSolder, symbol Device:C_Small
- added D3, D4, D5, D6, D7: LED, LED_SMD:LED_0805_2012Metric_Pad1.15x1.40mm_HandSolder, symbol Device:LED
- added J2: Conn_01x08, Connector_PinHeader_2.54mm:PinHeader_1x08_P2.54mm_Vertical, symbol Connector_Generic:Conn_01x08
- added R10: 1.5k, Resistor_SMD:R_0603_1608Metric_Pad1.05x0.95mm_HandSolder, symbol Device:R_Small
- added R11: 3.3k, Resistor_SMD:R_0603_1608Metric_Pad1.05x0.95mm_HandSolder, symbol Device:R_Small
- added R12: 47k, Resistor_SMD:R_0603_1608Metric_Pad1.05x0.95mm_HandSolder, symbol Device:R_Small
- added R13, R14, R15, R16, R6: 1k, Resistor_SMD:R_0603_1608Metric_Pad1.05x0.95mm_HandSolder, symbol Device:R_Small
- added R7: 1R, Resistor_SMD:R_1206_3216Metric_Pad1.42x1.75mm_HandSolder, symbol Device:R_Small
- added R8: 220, Resistor_SMD:R_0603_1608Metric_Pad1.05x0.95mm_HandSolder, symbol Device:R_Small
- added R9: 330, Resistor_SMD:R_0603_1608Metric_Pad1.05x0.95mm_HandSolder, symbol Device:R_Small
- added U3: MCP6L04x-xSL, Package_SO:SOIC-14_3.9x8.7mm_P1.27mm, symbol Amplifier_Operational:MCP6L04x-xSL
- R4, R5: value R_Small -> 400
Connections:
- net +3V3: now also R4.1, R5.1, J2.1 (Pin_1); no longer D1.2 (A), D2.2 (A)
- net DTR: now also J2.3 (Pin_3)
- net GND: now also C5.2, D3.1 (K), J2.6 (Pin_6), J2.7 (Pin_7), R12.2, U3.11 (V-)
- net PROG_RXD: now also J2.4 (Pin_4)
- net PROG_TXD: now also J2.5 (Pin_5)
- net RTS: now also J2.2 (Pin_2)
- net VBUS: now also C5.1, J2.8 (Pin_8), R13.2, R14.2, R15.2, R16.2, R6.2, R7.1, R8.1, U3.4 (V+); no longer C1.1, U1.3 (VI)
- net at U2.18 (~RXT~/GPIO.1): now also D2.1 (K); no longer R5.2
- net at U2.19 (~TXT~/GPIO.0): now also D1.1 (K); no longer R4.2
- new net: D1.2 (A), R4.2
- new net: D2.2 (A), R5.2
- new net: C1.1, R7.2, U1.3 (VI), U3.10 (+), U3.12 (+), U3.3 (+), U3.5 (+)
- new net: R11.2, R12.1, U3.6 (-)
- new net: R10.2, R11.1, U3.13 (-)
- new net: R10.1, R9.2, U3.9 (-)
- new net: R8.2, R9.1, U3.2 (-)
- new net: D4.1 (K), U3.1
- new net: D4.2 (A), R13.1
- new net: D5.1 (K), U3.8
- new net: D5.2 (A), R14.1
- new net: D6.1 (K), U3.14
- new net: D6.2 (A), R15.1
- new net: D7.1 (K), U3.7
- new net: D7.2 (A), R16.1
- new net: D3.2 (A), R6.1
Other:
- note added: "0,02V - 20mA"
- note added: "0,05V - 50mA"
- note added: "0,2V - 200mA"
- note added: "0,5V - 500mA"
- moved on the sheet: C1, C2, C3, C4, D1, D2, J1, L1, R1, R2, R3, R4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

Commit message: fab outputs for rev 2.0
Parts:
- R4, R5: value 400 -> 330
Changed lines of the file:
@@
 P 9300 3100
 F 0 "R4" H 9359 3146 50  0000 L CNN
-F 1 "400" H 9359 3055 50  0000 L CNN
+F 1 "330" H 9359 3055 50  0000 L CNN
 F 2 "Resistor_SMD:R_0603_1608Metric_Pad1.05x0.95mm_HandSolder" H 9300 3100 50  0001 C CNN
 F 3 "~" H 9300 3100 50  0001 C CNN
@@
 P 9700 3100
 F 0 "R5" H 9759 3146 50  0000 L CNN
-F 1 "400" H 9759 3055 50  0000 L CNN
+F 1 "330" H 9759 3055 50  0000 L CNN
 F 2 "Resistor_SMD:R_0603_1608Metric_Pad1.05x0.95mm_HandSolder" H 9700 3100 50  0001 C CNN
 F 3 "~" H 9700 3100 50  0001 C CNN
