File: lichtenprog.kicad_pcb (KiCad board)
At the start: 2 copper layers, 28 x 28 mm, 54 parts, among them J1 USB_C_Receptacle_USB2.0, J2 IO_OUT, U1 AZ1117-ADJ, U2 MCP6L04x-xSL, U3 USBLC6-2SC6, U4 CP2102N-A01-GQFN28, U5 SN74LVC1T45DBV, U6 SN74LVC1T45DBV

Commit message: some PCB swag, preparing JLC BOM
Parts:
- removed D8: 0.8V@100mA, Diode_SMD:D_SMA
- added C12: 10u, Capacitor_SMD:C_0603_1608Metric, F.Cu at (75.3, 64.5)
- added C13: 10u, Capacitor_SMD:C_0603_1608Metric, F.Cu at (68.8, 65.0)
- added R24: 10k, Resistor_SMD:R_0402_1005Metric, F.Cu at (73.5, 62.4)
- added R25: 22k, Resistor_SMD:R_0402_1005Metric, F.Cu at (76.9, 49.1)
- added R26: 1k, Resistor_SMD:R_0402_1005Metric, F.Cu at (71.7, 67.4)
- added SW1: VDD_RST, Button_Switch_SMD:SW_Push_1P1T_NO_Vertical_Wuerth_434133025816, F.Cu at (80.3, 48.3)
- added SW2: LIPO_RST, Button_Switch_SMD:SW_Push_1P1T_NO_Vertical_Wuerth_434133025816, F.Cu at (70.8, 70.8)
- added U7: SPX3819M5-L, Package_TO_SOT_SMD:SOT-23-5, F.Cu at (72.4, 64.5)
- C1: footprint Capacitor_SMD:C_0603_1608Metric -> Capacitor_SMD:C_0402_1005Metric
- JP1: footprint Jumper:SolderJumper-2_P1.3mm_Open_TrianglePad1.0x1.5mm -> Jumper:SolderJumper-2_P1.3mm_Bridged2Bar_Pad1.0x1.5mm
- JP4: value LIPO_SIMUL -> LIPO_EMUL_ENA; footprint Jumper:SolderJumper-2_P1.3mm_Bridged2Bar_Pad1.0x1.5mm -> Jumper:SolderJumper-3_P2.0mm_Open_TrianglePad1.0x1.5mm
- R12: value 47k -> 22k
- R13: value 0R -> 47k; footprint Resistor_SMD:R_1206_3216Metric_Pad1.30x1.75mm_HandSolder -> Resistor_SMD:R_0402_1005Metric
- R14: value 22.1k -> 22k
- R15: value 47.5k -> 47k
- R2: value 1R -> 2R/1206; footprint Resistor_SMD:R_1206_3216Metric_Pad1.30x1.75mm_HandSolder -> Resistor_SMD:R_1206_3216Metric
- R23: value DNP/1k -> 22k
- R5: value 220 -> 22k; footprint Resistor_SMD:R_0603_1608Metric_Pad0.98x0.95mm_HandSolder -> Resistor_SMD:R_0402_1005Metric
- R6: value 270 -> 47k; footprint Resistor_SMD:R_0603_1608Metric_Pad0.98x0.95mm_HandSolder -> Resistor_SMD:R_0402_1005Metric
- R7: value 100 -> 18k; footprint Resistor_SMD:R_0603_1608Metric_Pad0.98x0.95mm_HandSolder -> Resistor_SMD:R_0402_1005Metric
- R8: footprint Resistor_SMD:R_0603_1608Metric -> Resistor_SMD:R_0402_1005Metric
- U1: value AZ1117-ADJ -> SPX3819M5-L; footprint Package_TO_SOT_SMD:SOT-223-3_TabPin2 -> Package_TO_SOT_SMD:SOT-23-5
- moved R13 13.9 mm to (83.0, 51.4)
- moved JP1 11.3 mm to (71.4, 48.6), turned to -90 degrees
- moved R5 10.5 mm to (71.2, 47.7), turned to 180 degrees
- moved R6 9.95 mm to (73.3, 47.7), turned to 180 degrees
- moved R15 9.77 mm to (75.0, 61.9), turned to -90 degrees
- moved R7 9.48 mm to (75.3, 47.7), turned to 0 degrees
- moved R16 6.85 mm to (82.2, 55.2), turned to -90 degrees
- moved C2 4.60 mm to (75.3, 49.9), turned to 90 degrees
- moved R2 4.44 mm to (78.8, 51.4)
- moved R14 3.92 mm to (81.8, 51.4), turned to -90 degrees
- moved R8 2.24 mm to (81.6, 62.1), turned to 180 degrees
- moved U1 2.22 mm to (72.4, 49.9)
- moved JP4 2.14 mm to (71.4, 67.6), turned to 90 degrees
- moved R12 1.91 mm to (83.8, 68.4), turned to -90 degrees
- moved C3 1.71 mm to (72.5, 52.4)
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Connections:
- J1 pad A4: Net-(J1-PadA4) -> VBUS
- J1 pad A9: Net-(J1-PadA4) -> VBUS
- J1 pad B4: Net-(J1-PadA4) -> VBUS
- J1 pad B9: Net-(J1-PadA4) -> VBUS
- J2 pad 8: Net-(D8-Pad1) -> /VBUS_OUT
- JP4 pad 1: VBUS -> /VBUS_OUT
- JP4 pad 2: Net-(D8-Pad1) -> VBUS
- R13 pad 1: Net-(J1-PadA4) -> GND
- R13 pad 2: VBUS -> Net-(R13-Pad2)
- R14 pad 2: Net-(R14-Pad2) -> Net-(R13-Pad2)
- R15 pad 1: Net-(R14-Pad2) -> GND
- R15 pad 2: GND -> Net-(R15-Pad2)
- R23 pad 1: Net-(D8-Pad1) -> Net-(R23-Pad1)
- R23 pad 2: GND -> /VBUS_OUT
- R6 pad 1: Net-(JP1-Pad1) -> GND
- U1 pad 1: Net-(JP1-Pad2) -> Net-(C2-Pad1)
- U1 pad 2: VDD -> GND
- U1 pad 3: Net-(C2-Pad1) -> Net-(U1-Pad3)
- U2 pad 10: VBUS -> Net-(C2-Pad1)
- U2 pad 12: VBUS -> Net-(C2-Pad1)
- U2 pad 3: VBUS -> Net-(C2-Pad1)
- U2 pad 5: VBUS -> Net-(C2-Pad1)
- U3 pad 5: Net-(J1-PadA4) -> VBUS
- U4 pad 8: Net-(R14-Pad2) -> Net-(R13-Pad2)
Routing:
- net GND: track 32.5 -> 89.4 mm, vias 9 -> 26
- net Net-(C2-Pad1): track 0.00 -> 48.7 mm, vias 0 -> 3
- net VBUS: track 43.7 -> 67.6 mm, vias 4 -> 7
- net +3V3: track 32.0 -> 55.8 mm, vias 3 -> 6
- net Net-(J1-PadA4): track 14.0 -> 0.00 mm, vias 2 -> 0
- net Net-(R15-Pad2): track 0.00 -> 12.7 mm
- net /PROG_TX_3V3: track 20.2 -> 7.59 mm, vias 2 -> 1
- net /DTR: track 0.36 -> 12.9 mm, vias 0 -> 1
- net Net-(U1-Pad3): track 0.00 -> 10.5 mm, vias 0 -> 2
- net Net-(R13-Pad2): track 0.00 -> 9.57 mm
- net Net-(D1-Pad2): track 10.8 -> 1.64 mm, vias 1 -> 0
- net Net-(D4-Pad1): track 0.00 -> 7.67 mm
- net Net-(R10-Pad2): track 6.10 -> 13.6 mm
- net Net-(R14-Pad2): track 7.01 -> 0.00 mm
- net /VBUS_OUT: track 0.00 -> 4.78 mm
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- added copper zone on B.Cu, net /VBUS_OUT
- added copper zone on F.Cu, net /VBUS_OUT
- added copper zone on B.Cu, net GND
- added copper zone on F.Cu, net VBUS
Other:
- board text added: "3V3/~{1V8}"
- board text added: "Lichtenprog 4.0"
- board text added: "Rx pasthrough"
- board text added: "Rx translate"
- board text added: "Tx bypass"
- board text added: "Tx pasthrough"
- board text added: "VBUS pasthrough"
- board text added: "VBUS to v-lipo out"
- board text added: "github.com/cr1tbit/lichtenprog"
- board text added: "vdd rst"
- board text added: "vlipo rst"
- board text removed: "Lichtenprog rev 4.0 critbit @vcc.earth"

Commit message: repo cleanup before next rev
Parts:
- added H1: SCRHOLE, MountingHole:MountingHole_2.2mm_M2_ISO7380_Pad, F.Cu at (66.5, 71.5)
- added H2: SCRHOLE, MountingHole:MountingHole_2.2mm_M2_ISO7380_Pad, F.Cu at (89.5, 71.5)
- C5, C6: value 2u2 -> 2.2u
- R20, R22: value 470 -> 330
- R3, R4: value 470 -> 5.1k
- moved J2 0.25 mm to (65.5, 48.5)
Routing:
- net VDD: track 25.2 -> 25.7 mm
- net (no net): vias 2 -> 0
Other:
- board text added: "Tx translate"
- board text removed: "Tx bypass"

Commit message: route complt
Parts:
- removed C2, C3: 10u, Capacitor_SMD:C_0603_1608Metric
- removed D1, D2, D3, D4, D5, D6, D7: LED, LED_SMD:LED_0603_1608Metric
- removed JP2: RX_TRANS_BYPASS, Jumper:SolderJumper-3_P2.0mm_Open_TrianglePad1.0x1.5mm
- removed JP3: TX_TRANS_BYPASS, Jumper:SolderJumper-3_P2.0mm_Open_TrianglePad1.0x1.5mm
- removed JP4: LIPO_EMUL_ENA, Jumper:SolderJumper-3_P2.0mm_Open_TrianglePad1.0x1.5mm
- removed SW1: VDD_RST, Button_Switch_SMD:SW_Push_1P1T_NO_Vertical_Wuerth_434133025816
- removed SW2: LIPO_RST, Button_Switch_SMD:SW_Push_1P1T_NO_Vertical_Wuerth_434133025816
- removed U4: CP2102N-A01-GQFN28, Package_DFN_QFN:QFN-28-1EP_5x5mm_P0.5mm_EP3.35x3.35mm
- removed U6: SN74LVC1T45DBV, Package_TO_SOT_SMD:SOT-23-6
- removed U7: SPX3819M5-L, Package_TO_SOT_SMD:SOT-23-5
- added J3: USB_C_Receptacle_USB2.0, Connector_USB:USB_C_Receptacle_HRO_TYPE-C-31-M-12, F.Cu at (78.0, 48.9)
- added J4: Conn_02x08_Odd_Even, Connector_PinSocket_1.27mm:PinSocket_2x08_P1.27mm_Vertical_SMD, F.Cu at (87.0, 53.1)
- added J5: Conn_01x02, Connector_PinHeader_2.54mm:PinHeader_1x02_P2.54mm_Vertical, F.Cu at (68.0, 53.6)
- added L2: 2.2uH, Inductor_SMD:L_Sunlord_MWSA0412S, F.Cu at (69.3, 58.4)
- added LED1: XL-1606UGC, easyeda2kicad:LED-SMD_L1.7-W1.1-R-RD_GREEN, F.Cu at (91.2, 56.5)
- added LED10: XL-1606UGC, easyeda2kicad:LED-SMD_L1.7-W1.1-R-RD_GREEN, F.Cu at (71.3, 46.9)
- added LED11: XL-1606UGC, easyeda2kicad:LED-SMD_L1.7-W1.1-R-RD_GREEN, F.Cu at (89.0, 46.9)
- added LED2: XL-1606UGC, easyeda2kicad:LED-SMD_L1.7-W1.1-R-RD_GREEN, F.Cu at (91.2, 59.5)
- added LED3: XL-1606UGC, easyeda2kicad:LED-SMD_L1.7-W1.1-R-RD_GREEN, F.Cu at (91.2, 62.5)
- added LED4: XL-1606UGC, easyeda2kicad:LED-SMD_L1.7-W1.1-R-RD_GREEN, F.Cu at (91.2, 65.3)
- added LED5: XL-1606UGC, easyeda2kicad:LED-SMD_L1.7-W1.1-R-RD_GREEN, F.Cu at (91.2, 68.2)
- added LED6: XL-1606UGC, easyeda2kicad:LED-SMD_L1.7-W1.1-R-RD_GREEN, F.Cu at (84.5, 73.2)
- added LED7: XL-1606UGC, easyeda2kicad:LED-SMD_L1.7-W1.1-R-RD_GREEN, F.Cu at (91.2, 50.3)
- added LED8: XL-1606UGC, easyeda2kicad:LED-SMD_L1.7-W1.1-R-RD_GREEN, F.Cu at (91.2, 47.5)
- added LED9: XL-1606UGC, easyeda2kicad:LED-SMD_L1.7-W1.1-R-RD_GREEN, F.Cu at (68.7, 46.9)
- added R27: 5.1k, Resistor_SMD:R_0402_1005Metric, F.Cu at (75.1, 54.8)
- added R28: 5.1k, Resistor_SMD:R_0402_1005Metric, F.Cu at (82.9, 60.3)
- added R29: 1k, Resistor_SMD:R_0402_1005Metric, F.Cu at (89.6, 61.2)
- added R30: 22k, Resistor_SMD:R_0402_1005Metric, F.Cu at (76.6, 55.2)
- added R31: 22k, Resistor_SMD:R_0402_1005Metric, F.Cu at (77.6, 55.2)
- added TP1: TestPoint, TestPoint:TestPoint_Pad_D1.0mm, B.Cu at (85.6, 66.4)
- added TP2: TestPoint, TestPoint:TestPoint_Pad_D1.0mm, B.Cu at (87.1, 67.5)
- added TP3: TestPoint, TestPoint:TestPoint_Pad_D1.0mm, B.Cu at (91.2, 68.9)
- added TP4: TestPoint, TestPoint:TestPoint_Pad_D1.0mm, B.Cu at (91.2, 67.1)
- added U11: MT9700, easyeda2kicad:SOT-23-5_L3.0-W1.7-P0.95-LS2.8-BR, F.Cu at (70.7, 71.7)
- added U13: INA3221, Package_DFN_QFN:Texas_RGV0016A_VQFN-16-1EP_4x4mm_P0.65mm_EP2.1x2.1mm, F.Cu at (78.6, 58.8)
- added U15: USBLC6-4SC6, Package_TO_SOT_SMD:SOT-23-6, F.Cu at (79.8, 64.3)
- added U8: TLV62568DRL, Package_TO_SOT_SMD:SOT-563, F.Cu at (73.0, 55.6)
- added U9: MT9700, easyeda2kicad:SOT-23-5_L3.0-W1.7-P0.95-LS2.8-BR, F.Cu at (86.5, 60.5)
- added Y1: Crystal_GND24, Crystal:Crystal_SMD_3225-4Pin_3.2x2.5mm, F.Cu at (85.3, 70.1)
- C1: value 2.2u -> 10u; footprint Capacitor_SMD:C_0402_1005Metric -> Capacitor_SMD:C_0603_1608Metric
- C10: value 100n -> 10u; footprint Capacitor_SMD:C_0402_1005Metric -> Capacitor_SMD:C_0603_1608Metric
- C11, C9: value 100n -> 2.2u; footprint Capacitor_SMD:C_0402_1005Metric -> Capacitor_SMD:C_0603_1608Metric
- C12, C13: value 10u -> 100n; footprint Capacitor_SMD:C_0603_1608Metric -> Capacitor_SMD:C_0402_1005Metric
- C5, C6: footprint Capacitor_SMD:C_0402_1005Metric -> Capacitor_SMD:C_0603_1608Metric
- JP1: footprint Jumper:SolderJumper-2_P1.3mm_Bridged2Bar_Pad1.0x1.5mm -> Jumper:SolderJumper-2_P1.3mm_Open_RoundedPad1.0x1.5mm
- R1: value 1k -> 5.1k
- R10: value 1.5k -> 1k
- R11: value 3.3k -> 1k
- R12: value 22k -> 50mR/1206; footprint Resistor_SMD:R_0402_1005Metric -> Resistor_SMD:R_1206_3216Metric_Pad1.30x1.75mm_HandSolder
- R15: value 47k -> 50mR/1206; footprint Resistor_SMD:R_0402_1005Metric -> Resistor_SMD:R_1206_3216Metric_Pad1.30x1.75mm_HandSolder
- R16: value 1k -> 50mR/1206; footprint Resistor_SMD:R_0402_1005Metric -> Resistor_SMD:R_1206_3216Metric_Pad1.30x1.75mm_HandSolder
- R17, R19: value 1k -> 47k
- R18: value 1k -> 10k
- R2: value 2R/1206 -> 22k; footprint Resistor_SMD:R_1206_3216Metric -> Resistor_SMD:R_0402_1005Metric
- R20, R22: value 330 -> 22k
- R21, R26: value 1k -> 3k
- R24: value 10k -> 3k
- R25, R5: value 22k -> 3k
- R6: value 47k -> 3k
- R7: value 18k -> 3k
- R8: value 220 -> 47k
- R9: value 330 -> 1k
- U1: value SPX3819M5-L -> USBLC6-4SC6; footprint Package_TO_SOT_SMD:SOT-23-5 -> Package_TO_SOT_SMD:SOT-23-6
- U2: value MCP6L04x-xSL -> CH334F; footprint Package_SO:SOIC-14_3.9x8.7mm_P1.27mm -> easyeda2kicad:QFN-24_L4.0-W4.0-P0.50-BL-EP2.8
- U3: value USBLC6-2SC6 -> ~; footprint Package_TO_SOT_SMD:SOT-23-6 -> Critbit_lib:OLED_4Pin_128x64_new
- U5: value SN74LVC1T45DBV -> CP2102N-Axx-xQFN24; footprint Package_TO_SOT_SMD:SOT-23-6 -> Package_DFN_QFN:QFN-24-1EP_4x4mm_P0.5mm_EP2.6x2.6mm
- moved U3 75.0 mm to (132.5, 115.7)
- moved R1 25.9 mm to (86.6, 73.2), turned to 180 degrees
- moved R6 21.6 mm to (67.2, 68.4), turned to -90 degrees
- moved R26 20.7 mm to (66.9, 47.2), turned to 90 degrees
- moved R24 20.3 mm to (91.2, 52.5), turned to -90 degrees
- moved R5 17.9 mm to (83.9, 60.3), turned to -90 degrees
- moved R16 17.8 mm to (70.2, 68.3), turned to 180 degrees
- moved R17 17.4 mm to (74.2, 58.4)
- moved R19 15.7 mm to (75.2, 58.4)
- moved R18 15.4 mm to (75.5, 56.3), turned to 90 degrees
- moved R25 15.3 mm to (91.2, 54.4)
- moved R22 14.5 mm to (80.9, 62.0), turned to 180 degrees
- moved R15 14.0 mm to (70.0, 48.8), turned to 180 degrees
- moved C8 14.0 mm to (83.9, 66.3), turned to -90 degrees
- moved R13 13.0 mm to (74.2, 61.0)
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Connections:
- C1 pad 1: VBUS -> /HUB_3V3
- C12 pad 1: VBUS -> VDD
- C13 pad 1: /VBUS_OUT -> +3V3
- C8 pad 1: GND -> /HUB_3V3
- C8 pad 2: +3V3 -> GND
- C9 pad 1: GND -> VBUS
- C9 pad 2: +3V3 -> GND
- H1 pad 1: unconnected-(H1-Pad1) -> GND
- H2 pad 1: unconnected-(H2-Pad1) -> GND
- J1 pad A6: Net-(J1-PadA6) -> Net-(U15-I/O1)
- J1 pad A7: Net-(J1-PadA7) -> Net-(U15-I/O2)
- J1 pad B6: Net-(J1-PadA6) -> Net-(U15-I/O1)
- J1 pad B7: Net-(J1-PadA7) -> Net-(U15-I/O2)
- J2 pad 1: VDD -> /INA_VDDIO_RN
- J2 pad 2: /RTS -> /OUT_RTS
- J2 pad 3: /DTR -> /OUT_DTR
- J2 pad 4: /PROG_RX_VDD -> /OUT_RX
- J2 pad 5: /PROG_TX_VDD -> /OUT_TX
- J2 pad 8: /VBUS_OUT -> /INA_VBUSOUT_RN
- JP1 pad 1: Net-(JP1-Pad1) -> Net-(JP1-A)
- JP1 pad 2: Net-(JP1-Pad2) -> VDD
- R1 pad 1: Net-(D1-Pad2) -> GND
- R1 pad 2: VBUS -> Net-(LED6-K)
- R10 pad 1: Net-(R10-Pad1) -> Net-(LED3-K)
- R10 pad 2: Net-(R10-Pad2) -> /STAT_HUB_LED2
- R11 pad 1: Net-(R10-Pad2) -> VDD
- R11 pad 2: Net-(R11-Pad2) -> Net-(U5-~{RST})
- R12 pad 1: Net-(R11-Pad2) -> /INA_USBEXT_RP
- R12 pad 2: GND -> /INA_USBEXT_RN
- R13 pad 2: Net-(R13-Pad2) -> Net-(U5-VBUS)
- R14 pad 2: Net-(R13-Pad2) -> Net-(U5-VBUS)
- R15 pad 1: GND -> VDD
- R15 pad 2: Net-(R15-Pad2) -> /INA_VDDIO_RN
- R16 pad 1: +3V3 -> /INA_VBUSOUT_RP
- R16 pad 2: Net-(R16-Pad2) -> /INA_VBUSOUT_RN
- R17 pad 1: Net-(D2-Pad2) -> Net-(U8-FB)
- R17 pad 2: VBUS -> VDD
- R18 pad 1: Net-(D3-Pad2) -> GND
- R18 pad 2: VBUS -> Net-(U8-FB)
- R19 pad 1: Net-(D4-Pad2) -> Net-(U8-FB)
- R19 pad 2: VBUS -> Net-(JP1-A)
- R2 pad 1: VBUS -> /STAT_INA
- R2 pad 2: Net-(C2-Pad1) -> +3V3
- R20 pad 1: +3V3 -> /I2C_SDA
- R20 pad 2: Net-(D5-Pad2) -> +3V3
- R21 pad 1: Net-(D6-Pad2) -> /I2C_SCL
- R21 pad 2: VBUS -> +3V3
- R22 pad 1: +3V3 -> GND
- R23 pad 1: Net-(R23-Pad1) -> Net-(U13-PV)
- R23 pad 2: /VBUS_OUT -> +3V3
- R24 pad 1: GND -> Net-(LED7-A)
- R24 pad 2: Net-(R23-Pad1) -> +3V3
- R25 pad 1: Net-(C2-Pad1) -> Net-(LED8-A)
- R25 pad 2: Net-(R25-Pad2) -> +3V3
- R26 pad 1: Net-(JP4-Pad3) -> GND
- R26 pad 2: Net-(R15-Pad2) -> Net-(LED9-K)
- R5 pad 1: Net-(JP1-Pad2) -> GND
- R5 pad 2: VDD -> Net-(U9-SET)
- R6 pad 2: Net-(JP1-Pad2) -> Net-(U11-SET)
- R7 pad 1: GND -> /CTRL_VDDIO
- R7 pad 2: Net-(JP1-Pad1) -> VBUS
- R8 pad 1: VBUS -> GND
- R8 pad 2: Net-(R8-Pad2) -> Net-(U2-PSELF)
- R9 pad 1: Net-(R8-Pad2) -> Net-(LED1-K)
- R9 pad 2: Net-(R10-Pad1) -> /STAT_HUB_LED1
- U1 pad 1: Net-(C2-Pad1) -> /OUT_RTS
- U1 pad 3: Net-(R25-Pad2) -> /OUT_DTR
- U1 pad 4: Net-(JP1-Pad2) -> /OUT_RX
- U1 pad 5: VDD -> VBUS
- U2 pad 10: Net-(C2-Pad1) -> /MCU_DP
- U2 pad 11: GND -> /OUT_DM
- U2 pad 12: Net-(C2-Pad1) -> /OUT_DP
- U2 pad 13: Net-(R10-Pad2) -> /STAT_HUB_LED3
- U2 pad 14: Net-(D4-Pad1) -> Net-(U15-I/O2)
- U2 pad 2: Net-(R8-Pad2) -> unconnected-(U2-NC.-Pad2)
- U2 pad 3: Net-(C2-Pad1) -> Net-(U2-XO)
- U2 pad 4: VBUS -> Net-(U2-XI)
- U2 pad 5: Net-(C2-Pad1) -> /CP_DM
- U2 pad 6: Net-(R11-Pad2) -> /CP_DP
- U2 pad 9: Net-(R10-Pad1) -> /MCU_DM
- U3 pad 1: Net-(J1-PadA6) -> unconnected-(U3-GND-Pad1)
- U3 pad 2: GND -> unconnected-(U3-VCC-Pad2)
- U3 pad 3: Net-(J1-PadA7) -> unconnected-(U3-SCL-Pad3)
- U3 pad 4: Net-(U3-Pad4) -> unconnected-(U3-SDA-Pad4)
- U5 pad 1: +3V3 -> unconnected-(U5-~{RI}/CLK-Pad1)
- U5 pad 3: /PROG_TX_3V3 -> /CP_DP
- U5 pad 4: Net-(JP3-Pad3) -> /CP_DM
- U5 pad 5: +3V3 -> VDD
- U5 pad 6: VDD -> +3V3
Routing:
- net Net-(C2-Pad1): track 48.7 -> 0.00 mm, vias 3 -> 0
- net /STAT_LED_TX: track 0.00 -> 45.3 mm, vias 0 -> 2
- net /STAT_LED_RX: track 0.00 -> 42.8 mm, vias 0 -> 2
- net /CTRL_VBUSOUT: track 0.00 -> 39.5 mm, vias 0 -> 2
- net /OUT_DM: track 0.00 -> 36.2 mm, vias 0 -> 3
- net /INA_VBUSOUT_RP: track 0.00 -> 35.9 mm, vias 0 -> 3
- net +3V3: track 55.8 -> 20.6 mm, vias 6 -> 7
- net VDD: track 25.7 -> 59.1 mm, vias 0 -> 2
- net /OUT_DP: track 0.00 -> 32.8 mm, vias 0 -> 3
- net /OUT_TX: track 0.00 -> 31.1 mm, vias 0 -> 3
- net /CTRL_VDDIO: track 0.00 -> 26.9 mm, vias 0 -> 2
- net /INA_USBEXT_RN: track 0.00 -> 24.7 mm, vias 0 -> 2
- net /OUT_RX: track 0.00 -> 22.8 mm, vias 0 -> 2
- net /INA_VBUSOUT_RN: track 0.00 -> 20.8 mm, vias 0 -> 2
- net Net-(LED11-A): track 0.00 -> 20.4 mm, vias 0 -> 2
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- added copper zone on In1.Cu, net +3V3
- added copper zone on In2.Cu, net GND
- added copper zone on In1.Cu, net VBUS
- removed copper zone on B.Cu, net /VBUS_OUT
- removed copper zone on F.Cu, net /VBUS_OUT
- removed copper zone on B.Cu, net GND
- removed copper zone on F.Cu, net VBUS
Other:
- outline, holes or cut-outs redrawn
- copper layers 2 -> 4
- board text added: "1V8"
- board text added: "DM"
- board text added: "DP"
- board text added: "OVC"
- board text added: "PWR"
- board text removed: "200mA"
- board text removed: "20mA"
- board text removed: "500mA"
- board text removed: "50mA"
- board text removed: "vlipo rst"
